Commit message: [everything] Fixes here and there for the demo

File: resources/objects/apartment.urdf (robot description, URDF)
Before this commit: robot apartment, 113 links, 112 joints
Links:
- removed link cabinet1
- removed link cabinet10
- removed link cabinet10_drawer_bottom
- removed link cabinet10_drawer_middle
- removed link cabinet10_drawer_top
- removed link cabinet11
- removed link cabinet11_drawer_bottom
- removed link cabinet11_drawer_middle
- removed link cabinet11_drawer_top
- removed link cabinet1_coloksu_level4
- removed link cabinet1_coloksu_level5
- removed link cabinet1_door_top_left
- removed link cabinet1_drawer_bottom
- removed link cabinet1_drawer_middle
- removed link cabinet2
- removed link cabinet2_door_left
- removed link cabinet2_door_out_fancy
- removed link cabinet2_drawer_big
- removed link cabinet2_drawer_small
- removed link cabinet3
- removed link cabinet3_door_bottom_left
- removed link cabinet3_door_bottom_out_fancy
- removed link cabinet3_door_top_left
- removed link cabinet3_door_top_out_fancy
- removed link cabinet4
- removed link cabinet4_door_bottom
- removed link cabinet4_door_top
- removed link cabinet5
- removed link cabinet5_drawer_bottom
- removed link cabinet5_drawer_middle
- removed link cabinet5_drawer_top
- removed link cabinet6
- removed link cabinet6_drawer_bottom
- removed link cabinet6_drawer_middle
- removed link cabinet6_drawer_top
- removed link cabinet7
- removed link cabinet7_door_bottom_left
- removed link cabinet8
- removed link cabinet8_drawer_bottom
- removed link cabinet8_drawer_middle
- removed link cabinet9
- removed link cabinet9_drawer_bottom
- removed link cabinet9_drawer_middle
- removed link cabinet9_drawer_top
- removed link dishwasher_drawer_middle
- removed link handle_cab10_b
- removed link handle_cab10_m
- removed link handle_cab10_t
- removed link handle_cab11_b
- removed link handle_cab11_m
- removed link handle_cab11_t
- removed link handle_cab1_drawer_bottom
- removed link handle_cab1_drawer_mid
- removed link handle_cab1_top_door
- removed link handle_cab2_door
- removed link handle_cab3_door_bottom
- removed link handle_cab3_door_top
- removed link handle_cab4_door_bottom
- removed link handle_cab5_b
- removed link handle_cab5_m
- removed link handle_cab5_t
- removed link handle_cab6_b
- removed link handle_cab6_m
- removed link handle_cab6_t
- removed link handle_cab7
- removed link handle_cab7_middle
- removed link handle_cab8
- removed link handle_cab9_b
- removed link handle_cab9_m
- removed link handle_cab9_t
- removed link table_area_main
- added link coffee_area_bottom_left; collision mesh filename=package://iai_apartment/meshes/cabinet05/IAIKitchenCabinet5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; visual mesh filename=package://iai_apartment/meshes/cabinet05/IAIKitchenCabinet5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
- added link coffee_area_bottom_left_bottom_drawer; collision mesh filename=package://iai_apartment/meshes/cabinet05/IAIKitchenDrawerW6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; visual mesh filename=package://iai_apartment/meshes/cabinet05/IAIKitchenDrawerW6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
- added link coffee_area_bottom_left_bottom_handle; collision mesh filename=package://iai_apartment/meshes/handles/handle_horizontal.obj; visual mesh filename=package://iai_apartment/meshes/handles/handle_horizontal.dae
- added link coffee_area_bottom_left_middle_drawer; collision mesh filename=package://iai_apartment/meshes/cabinet05/IAIKitchenDrawerW6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; visual mesh filename=package://iai_apartment/meshes/cabinet05/IAIKitchenDrawerW6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
- added link coffee_area_bottom_left_middle_handle; collision mesh filename=package://iai_apartment/meshes/handles/handle_horizontal.obj; visual mesh filename=package://iai_apartment/meshes/handles/handle_horizontal.dae
- added link coffee_area_bottom_left_top_drawer; collision mesh filename=package://iai_apartment/meshes/cabinet05/IAIKitchenDrawerW6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; visual mesh filename=package://iai_apartment/meshes/cabinet05/IAIKitchenDrawerW6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
- added link coffee_area_bottom_left_top_handle; collision mesh filename=package://iai_apartment/meshes/handles/handle_horizontal.obj; visual mesh filename=package://iai_apartment/meshes/handles/handle_horizontal.dae
- added link coffee_area_bottom_right; collision mesh filename=package://iai_apartment/meshes/cabinet06/IAIKitchenCabinet6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; visual mesh filename=package://iai_apartment/meshes/cabinet06/IAIKitchenCabinet6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
- added link coffee_area_bottom_right_bottom_drawer; collision mesh filename=package://iai_apartment/meshes/cabinet06/IAIKitchenDrawerW4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; visual mesh filename=package://iai_apartment/meshes/cabinet06/IAIKitchenDrawerW4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
- added link coffee_area_bottom_right_bottom_handle; collision mesh filename=package://iai_apartment/meshes/handles/handle_horizontal.obj; visual mesh filename=package://iai_apartment/meshes/handles/handle_horizontal.dae
- added link coffee_area_bottom_right_middle_drawer; collision mesh filename=package://iai_apartment/meshes/cabinet06/IAIKitchenDrawerW4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; visual mesh filename=package://iai_apartment/meshes/cabinet06/IAIKitchenDrawerW4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
- added link coffee_area_bottom_right_middle_handle; collision mesh filename=package://iai_apartment/meshes/handles/handle_horizontal.obj; visual mesh filename=package://iai_apartment/meshes/handles/handle_horizontal.dae
- added link coffee_area_bottom_right_top_drawer; collision mesh filename=package://iai_apartment/meshes/cabinet06/IAIKitchenDrawerW4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; visual mesh filename=package://iai_apartment/meshes/cabinet06/IAIKitchenDrawerW4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
- added link coffee_area_bottom_right_top_handle; collision mesh filename=package://iai_apartment/meshes/handles/handle_horizontal.obj; visual mesh filename=package://iai_apartment/meshes/handles/handle_horizontal.dae
- added link coffee_area_top; collision mesh filename=package://iai_apartment/meshes/cabinet04/IAIKitchenCabinet4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; visual mesh filename=package://iai_apartment/meshes/cabinet04/IAIKitchenCabinet4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
- added link coffee_area_top_door_bottom; collision mesh filename=package://iai_apartment/meshes/cabinet04/IAIDoor2W100H40.obj; visual mesh filename=package://iai_apartment/meshes/cabinet04/IAIDoor2W100H40.dae
- added link coffee_area_top_door_top; collision mesh filename=package://iai_apartment/meshes/cabinet04/IAIDoor1W100H40.obj; visual mesh filename=package://iai_apartment/meshes/cabinet04/IAIDoor1W100H40.dae
- added link coffee_area_top_handle; collision mesh filename=package://iai_apartment/meshes/handles/handle_horizontal.obj; visual mesh filename=package://iai_apartment/meshes/handles/handle_horizontal.dae
- added link dishwasher; collision mesh filename=package://iai_apartment/meshes/cabinet07/IAIKitchenCabinet7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; visual mesh filename=package://iai_apartment/meshes/cabinet07/IAIKitchenCabinet7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
- added link dishwasher_door; collision mesh filename=package://iai_apartment/meshes/cabinet07/IAIKitchenDoorW60H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; visual mesh filename=package://iai_apartment/meshes/cabinet07/IAIKitchenDoorW60H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
- added link dishwasher_door_handle; collision mesh filename=package://iai_apartment/meshes/handles/handle_horizontal.obj; visual mesh filename=package://iai_apartment/meshes/handles/handle_horizontal.dae
- added link dishwasher_drawer; collision mesh filename=package://iai_apartment/meshes/cabinet07/dishwasher_drawer_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; visual mesh filename=package://iai_apartment/meshes/cabinet07/dishwasher_drawer_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
- added link dishwasher_drawer_handle; collision box size=0.015 0.325 0.021; visual box size=0.015 0.325 0.021
- added link fridge_area; collision mesh filename=package://iai_apartment/meshes/cabinet03/IAICabinet3W60.obj; visual mesh filename=package://iai_apartment/meshes/cabinet03/IAICabinet3W60.dae
- added link fridge_area_bottom_door; collision mesh filename=package://iai_apartment/meshes/cabinet03/IAIDoorW60H80.obj; visual mesh filename=package://iai_apartment/meshes/cabinet03/IAIDoorW60H80.dae
- added link fridge_area_bottom_door_handle; collision mesh filename=package://iai_apartment/meshes/handles/handle_horizontal.obj; visual mesh filename=package://iai_apartment/meshes/handles/handle_horizontal.dae
- added link fridge_area_door_bottom_out_fancy
- added link fridge_area_door_top_out_fancy
- added link fridge_area_top_door; collision mesh filename=package://iai_apartment/meshes/cabinet03/IAIDoorW60H133.obj; visual mesh filename=package://iai_apartment/meshes/cabinet03/IAIDoorW60H133.dae
- added link fridge_area_top_door_handle; collision mesh filename=package://iai_apartment/meshes/handles/handle_horizontal.obj; visual mesh filename=package://iai_apartment/meshes/handles/handle_horizontal.dae
- added link fridge_back; collision box size=0.036 0.56 1.2; visual box size=0.036 0.56 1.2
- added link fridge_bottom_side; collision box size=0.5 0.535 0.036; visual box size=0.5 0.535 0.036
- added link fridge_left_side; collision box size=0.036 0.5 1.2; visual box size=0.036 0.5 1.2
- added link fridge_level1; collision box size=0.5 0.535 0.036; visual box size=0.5 0.535 0.036
- added link fridge_main
- added link fridge_right_side; collision box size=0.036 0.5 1.2; visual box size=0.036 0.5 1.2
- added link fridge_top_side; collision box size=0.5 0.535 0.036; visual box size=0.5 0.535 0.036
- added link island_left; collision mesh filename=package://iai_apartment/meshes/cabinet09/IAIKitchenCabinet9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; visual mesh filename=package://iai_apartment/meshes/cabinet09/IAIKitchenCabinet9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
- added link island_left_bottom_handle; collision mesh filename=package://iai_apartment/meshes/handles/handle_horizontal.obj; visual mesh filename=package://iai_apartment/meshes/handles/handle_horizontal.dae
- added link island_left_drawer_bottom; collision mesh filename=package://iai_apartment/meshes/cabinet09/IAIKitchenDrawerW6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; visual mesh filename=package://iai_apartment/meshes/cabinet09/IAIKitchenDrawerW6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
- added link island_left_drawer_middle; collision mesh filename=package://iai_apartment/meshes/cabinet09/IAIKitchenDrawerW6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; visual mesh filename=package://iai_apartment/meshes/cabinet09/IAIKitchenDrawerW6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
- added link island_left_drawer_top; collision mesh filename=package://iai_apartment/meshes/cabinet09/IAIKitchenDrawerW6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; visual mesh filename=package://iai_apartment/meshes/cabinet09/IAIKitchenDrawerW6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
- added link island_left_middle_handle; collision mesh filename=package://iai_apartment/meshes/handles/handle_horizontal.obj; visual mesh filename=package://iai_apartment/meshes/handles/handle_horizontal.dae
- added link island_left_top_handle; collision mesh filename=package://iai_apartment/meshes/handles/handle_horizontal.obj; visual mesh filename=package://iai_apartment/meshes/handles/handle_horizontal.dae
- added link island_middle; collision mesh filename=package://iai_apartment/meshes/cabinet10/IAIKitchenCabinet9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; visual mesh filename=package://iai_apartment/meshes/cabinet10/IAIKitchenCabinet9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
- added link island_middle_bottom_handle; collision mesh filename=package://iai_apartment/meshes/handles/handle_horizontal.obj; visual mesh filename=package://iai_apartment/meshes/handles/handle_horizontal.dae
- added link island_middle_drawer_bottom; collision mesh filename=package://iai_apartment/meshes/cabinet10/IAIKitchenDrawerW4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; visual mesh filename=package://iai_apartment/meshes/cabinet10/IAIKitchenDrawerW4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
- added link island_middle_drawer_middle; collision mesh filename=package://iai_apartment/meshes/cabinet10/IAIKitchenDrawerW4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; visual mesh filename=package://iai_apartment/meshes/cabinet10/IAIKitchenDrawerW4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
- added link island_middle_drawer_top; collision mesh filename=package://iai_apartment/meshes/cabinet10/IAIKitchenDrawerW4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; visual mesh filename=package://iai_apartment/meshes/cabinet10/IAIKitchenDrawerW4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
- added link island_middle_middle_handle; collision mesh filename=package://iai_apartment/meshes/handles/handle_horizontal.obj; visual mesh filename=package://iai_apartment/meshes/handles/handle_horizontal.dae
- added link island_middle_top_handle; collision mesh filename=package://iai_apartment/meshes/handles/handle_horizontal.obj; visual mesh filename=package://iai_apartment/meshes/handles/handle_horizontal.dae
- added link island_right; collision mesh filename=package://iai_apartment/meshes/cabinet11/IAIKitchenCabinet1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; visual mesh filename=package://iai_apartment/meshes/cabinet11/IAIKitchenCabinet1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
- added link island_right_bottom_handle; collision mesh filename=package://iai_apartment/meshes/handles/handle_horizontal.obj; visual mesh filename=package://iai_apartment/meshes/handles/handle_horizontal.dae
- added link island_right_drawer_bottom; collision mesh filename=package://iai_apartment/meshes/cabinet11/IAIKitchenDrawerW9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; visual mesh filename=package://iai_apartment/meshes/cabinet11/IAIKitchenDrawerW9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
- added link island_right_drawer_middle; collision mesh filename=package://iai_apartment/meshes/cabinet11/IAIKitchenDrawerW9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; visual mesh filename=package://iai_apartment/meshes/cabinet11/IAIKitchenDrawerW9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
- added link island_right_drawer_top; collision mesh filename=package://iai_apartment/meshes/cabinet11/IAIKitchenDrawerW9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; visual mesh filename=package://iai_apartment/meshes/cabinet11/IAIKitchenDrawerW9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
- added link island_right_middle_handle; collision mesh filename=package://iai_apartment/meshes/handles/handle_horizontal.obj; visual mesh filename=package://iai_apartment/meshes/handles/handle_horizontal.dae
- added link island_right_top_handle; collision mesh filename=package://iai_apartment/meshes/handles/handle_horizontal.obj; visual mesh filename=package://iai_apartment/meshes/handles/handle_horizontal.dae
- added link oven_area; collision mesh filename=package://iai_apartment/meshes/cabinet01/IAICabinet1W60.obj; visual mesh filename=package://iai_apartment/meshes/cabinet01/IAICabinet1W60.dae
- added link oven_area_coloksu_level4; collision box size=0.534 0.568 0.003; visual box size=0.534 0.568 0.003
- added link oven_area_coloksu_level5; collision box size=0.534 0.568 0.02; visual box size=0.534 0.568 0.02
- added link oven_area_door_top_left; collision mesh filename=package://iai_apartment/meshes/cabinet01/IAIDoorW60H80.obj; visual mesh filename=package://iai_apartment/meshes/cabinet01/IAIDoorW60H80.dae
- added link oven_area_door_top_left_handle; collision mesh filename=package://iai_apartment/meshes/handles/handle_horizontal.obj; visual mesh filename=package://iai_apartment/meshes/handles/handle_horizontal.dae
- added link oven_area_drawer_bottom; collision mesh filename=package://iai_apartment/meshes/cabinet01/IAIDrawerW60H53.obj; visual mesh filename=package://iai_apartment/meshes/cabinet01/IAIDrawerW60H53.dae
- added link oven_area_drawer_bottom_handle; collision mesh filename=package://iai_apartment/meshes/handles/handle_horizontal.obj; visual mesh filename=package://iai_apartment/meshes/handles/handle_horizontal.dae
- added link oven_area_drawer_middle; collision mesh filename=package://iai_apartment/meshes/cabinet01/IAIDrawerW60H26.obj; visual mesh filename=package://iai_apartment/meshes/cabinet01/IAIDrawerW60H26.dae
- added link oven_area_drawer_middle_handle; collision mesh filename=package://iai_apartment/meshes/handles/handle_horizontal.obj; visual mesh filename=package://iai_apartment/meshes/handles/handle_horizontal.dae
- added link oven_area_left; collision mesh filename=package://iai_apartment/meshes/cabinet12/IAICabinet12W60.obj; visual mesh filename=package://iai_apartment/meshes/cabinet12/IAICabinet12W60.dae
- added link oven_area_left_door_bottom_left; collision mesh filename=package://iai_apartment/meshes/cabinet12/IAIDoorW60H80.obj; visual mesh filename=package://iai_apartment/meshes/cabinet12/IAIDoorW60H80.dae
- added link oven_area_left_door_bottom_out_fancy
- added link oven_area_left_door_top; collision mesh filename=package://iai_apartment/meshes/cabinet12/IAIDoorW60H133.obj; visual mesh filename=package://iai_apartment/meshes/cabinet12/IAIDoorW60H133.dae
- added link oven_area_left_door_top_out_fancy
- added link oven_area_right; collision mesh filename=package://iai_apartment/meshes/cabinet02/IAICabinet2W40H57.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; visual mesh filename=package://iai_apartment/meshes/cabinet02/IAICabinet2W40H57.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
- added link oven_area_right_door; collision mesh filename=package://iai_apartment/meshes/cabinet02/IAIDoorW40H212.obj; visual mesh filename=package://iai_apartment/meshes/cabinet02/IAIDoorW40H212.dae
- added link oven_area_right_door_out_fancy
- added link oven_area_right_drawer_big; collision mesh filename=package://iai_apartment/meshes/cabinet02/IAIDrawerW40H22.obj; visual mesh filename=package://iai_apartment/meshes/cabinet02/IAIDrawerW40H22.dae
- added link oven_area_right_drawer_small; collision mesh filename=package://iai_apartment/meshes/cabinet02/IAIDrawerW40H10.obj; visual mesh filename=package://iai_apartment/meshes/cabinet02/IAIDrawerW40H10.dae
- added link oven_area_right_handle; collision mesh filename=package://iai_apartment/meshes/handles/handle_horizontal.obj; visual mesh filename=package://iai_apartment/meshes/handles/handle_horizontal.dae
- added link sink_area; collision mesh filename=package://iai_apartment/meshes/cabinet08/IAIKitchenCabinet8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; visual mesh filename=package://iai_apartment/meshes/cabinet08/IAIKitchenCabinet8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
- added link sink_area_drawer_bottom; collision mesh filename=package://iai_apartment/meshes/cabinet08/IAIKitchenDrawerW6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; visual mesh filename=package://iai_apartment/meshes/cabinet08/IAIKitchenDrawerW6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
- added link sink_area_drawer_middle; collision mesh filename=package://iai_apartment/meshes/cabinet08/IAIKitchenDrawerW5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; visual mesh filename=package://iai_apartment/meshes/cabinet08/IAIKitchenDrawerW5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
- added link sink_area_handle; collision mesh filename=package://iai_apartment/meshes/handles/handle_horizontal.obj; visual mesh filename=package://iai_apartment/meshes/handles/handle_horizontal.dae
Joints:
- removed joint cabinet10_drawer_bottom_joint
- removed joint cabinet10_drawer_middle_joint
- removed joint cabinet10_drawer_top_joint
- removed joint cabinet10_joint
- removed joint cabinet11_drawer_bottom_joint
- removed joint cabinet11_drawer_middle_joint
- removed joint cabinet11_drawer_top_joint
- removed joint cabinet11_joint
- removed joint cabinet1_coloksu_level4_joint
- removed joint cabinet1_coloksu_level5_joint
- removed joint cabinet1_door_top_left_joint
- removed joint cabinet1_drawer_bottom_joint
- removed joint cabinet1_drawer_middle_joint
- removed joint cabinet1_joint
- removed joint cabinet2_door_left_joint
- removed joint cabinet2_door_out_joint
- removed joint cabinet2_drawer_big_joint
- removed joint cabinet2_drawer_small_joint
- removed joint cabinet2_joint
- removed joint cabinet3_door_bottom_left_joint
- removed joint cabinet3_door_bottom_out_joint
- removed joint cabinet3_door_top_left_joint
- removed joint cabinet3_door_top_out_joint
- removed joint cabinet3_joint
- removed joint cabinet4_door_bottom_bottom_joint
- removed joint cabinet4_door_top_top_joint
- removed joint cabinet4_joint
- removed joint cabinet5_drawer_bottom_joint
- removed joint cabinet5_drawer_middle_joint
- removed joint cabinet5_drawer_top_joint
- removed joint cabinet5_joint
- removed joint cabinet6_drawer_bottom_joint
- removed joint cabinet6_drawer_middle_joint
- removed joint cabinet6_drawer_top_joint
- removed joint cabinet6_joint
- removed joint cabinet7_door_bottom_left_joint
- removed joint cabinet7_joint
- removed joint cabinet8_drawer_bottom_joint
- removed joint cabinet8_drawer_middle_joint
- removed joint cabinet8_joint
- removed joint cabinet9_drawer_bottom_joint
- removed joint cabinet9_drawer_middle_joint
- removed joint cabinet9_drawer_top_joint
- removed joint cabinet9_joint
- removed joint handle_cab10_bott_joint
- removed joint handle_cab10_mid_joint
- removed joint handle_cab10_top_joint
- removed joint handle_cab11_bott_joint
- removed joint handle_cab11_mid_joint
- removed joint handle_cab11_top_joint
- removed joint handle_cab1_drawer_bottom_joint
- removed joint handle_cab1_drawer_mid_joint
- removed joint handle_cab1_top_door_joint
- removed joint handle_cab3_door_bottom_joint
- removed joint handle_cab3_door_top_joint
- removed joint handle_cab4_door_bottom_joint
- removed joint handle_cab5_bott_joint
- removed joint handle_cab5_mid_joint
- removed joint handle_cab5_top_joint
- removed joint handle_cab6_bott_joint
- removed joint handle_cab6_mid_joint
- removed joint handle_cab6_top_joint
- removed joint handle_cab7_drawer_middle_joint
- removed joint handle_cab7_top_joint
- removed joint handle_cab8_top_joint
- removed joint handle_cab9_bott_joint
- removed joint handle_cab9_mid_joint
- removed joint handle_cab9_top_joint
- removed joint table_area_main_joint
- added joint coffee_area_bottom_left_bottom_drawer_joint: type prismatic, parent coffee_area_bottom_left, child coffee_area_bottom_left_bottom_drawer, origin xyz=0.037 0.0 -0.28 rpy=0 0 3.14, axis -1 0 0, limit lower=0.0 upper=0.45 effort=1000.0 velocity=0.5
- added joint coffee_area_bottom_left_bottom_handle_joint: type fixed, parent coffee_area_bottom_left_bottom_drawer, child coffee_area_bottom_left_bottom_handle, origin xyz=-0.235 0 0.245 rpy=1.57 0 0
- added joint coffee_area_bottom_left_joint: type fixed, parent side_A, child coffee_area_bottom_left, origin xyz=-0.121 1.625 0.4
- added joint coffee_area_bottom_left_middle_drawer_joint: type prismatic, parent coffee_area_bottom_left, child coffee_area_bottom_left_middle_drawer, origin xyz=0.027 0.0 0.107 rpy=0 0 3.14, axis -1 0 0, limit lower=0.0 upper=0.45 effort=1000.0 velocity=0.5
- added joint coffee_area_bottom_left_middle_handle_joint: type fixed, parent coffee_area_bottom_left_middle_drawer, child coffee_area_bottom_left_middle_handle, origin xyz=-0.245 0 0.13 rpy=1.57 0 0
- added joint coffee_area_bottom_left_top_drawer_joint: type prismatic, parent coffee_area_bottom_left, child coffee_area_bottom_left_top_drawer, origin xyz=0.03 0.0 0.327 rpy=0 0 3.14, axis -1 0 0, limit lower=0.0 upper=0.45 effort=1000.0 velocity=0.5
- added joint coffee_area_bottom_left_top_handle_joint: type fixed, parent coffee_area_bottom_left_top_drawer, child coffee_area_bottom_left_top_handle, origin xyz=-0.245 0 0.05 rpy=1.57 0 0
- added joint coffee_area_bottom_right_bottom_drawer_joint: type prismatic, parent coffee_area_bottom_right, child coffee_area_bottom_right_bottom_drawer, origin xyz=0.047 0.0 -0.28 rpy=0 0 3.14, axis -1 0 0, limit lower=0.0 upper=0.45 effort=1000.0 velocity=0.5
- added joint coffee_area_bottom_right_bottom_handle_joint: type fixed, parent coffee_area_bottom_right_bottom_drawer, child coffee_area_bottom_right_bottom_handle, origin xyz=-0.227 0 0.245 rpy=1.57 0 0
- added joint coffee_area_bottom_right_joint: type fixed, parent side_A, child coffee_area_bottom_right, origin xyz=-0.121 2.127 0.4
- added joint coffee_area_bottom_right_middle_drawer_joint: type prismatic, parent coffee_area_bottom_right, child coffee_area_bottom_right_middle_drawer, origin xyz=0.03 0.0 0.105 rpy=0 0 3.14, axis -1 0 0, limit lower=0.0 upper=0.45 effort=1000.0 velocity=0.5
- added joint coffee_area_bottom_right_middle_handle_joint: type fixed, parent coffee_area_bottom_right_middle_drawer, child coffee_area_bottom_right_middle_handle, origin xyz=-0.245 0 0.13 rpy=1.57 0 0
- added joint coffee_area_bottom_right_top_drawer_joint: type prismatic, parent coffee_area_bottom_right, child coffee_area_bottom_right_top_drawer, origin xyz=0.033 -0.0125 0.328 rpy=0 0 3.14, axis -1 0 0, limit lower=0.0 upper=0.45 effort=1000.0 velocity=0.5
- added joint coffee_area_bottom_right_top_handle_joint: type fixed, parent coffee_area_bottom_right_top_drawer, child coffee_area_bottom_right_top_handle, origin xyz=-0.238 0 0.05 rpy=1.57 0 0
- added joint coffee_area_top_door_bottom_bottom_joint: type revolute, parent coffee_area_top_door_top, child coffee_area_top_door_bottom, origin xyz=0.0 0.0 -0.4 rpy=0 0 0, axis 0 -1 0, limit lower=0.0 upper=1.5708 effort=1000.0 velocity=1.5708, mimic joint=coffee_area_top_door_top_top_joint multiplier=1.2
- added joint coffee_area_top_door_top_top_joint: type revolute, parent coffee_area_top, child coffee_area_top_door_top, origin xyz=0.07 0 0.42 rpy=0 0 3.14, axis 0 1 0, limit lower=0 upper=2.0 effort=1000.0 velocity=1.5708
- added joint coffee_area_top_handle_joint: type fixed, parent coffee_area_top_door_bottom, child coffee_area_top_handle, origin xyz=-0.055 0 -0.35 rpy=1.57 0 0
- added joint coffee_area_top_joint: type fixed, parent side_A, child coffee_area_top, origin xyz=-0.175 1.825 1.72
- added joint dishwasher_door_bottom_left_joint: type revolute, parent dishwasher, child dishwasher_door, origin xyz=0.372 0 -0.45 rpy=0 0 3.14, axis 0 -1 0, limit lower=0.0 upper=1.5708 effort=1000.0 velocity=1.5708
- added joint dishwasher_drawer_middle_handle_joint: type fixed, parent dishwasher_drawer, child dishwasher_drawer_handle, origin xyz=-0.315 0 0.068 rpy=1.57 0 0
- added joint dishwasher_handle_top_joint: type fixed, parent dishwasher_door, child dishwasher_door_handle, origin xyz=-0.06 0 0.74 rpy=1.57 0 0
- added joint dishwasher_joint: type fixed, parent side_B, child dishwasher, origin xyz=0.2 0.501 0.47
- added joint fridge_area_door_bottom_left_handle_joint: type fixed, parent fridge_area_bottom_door, child fridge_area_bottom_door_handle, origin xyz=-0.036 -0.45 0.1 rpy=1.57 0 0
- added joint fridge_area_door_bottom_left_joint: type revolute, parent fridge_area_door_bottom_out_fancy, child fridge_area_bottom_door, axis 0 0 -1, limit lower=0.0 upper=1.5708 effort=1000.0 velocity=1.5708
- added joint fridge_area_door_bottom_out_joint: type prismatic, parent fridge_area, child fridge_area_door_bottom_out_fancy, origin xyz=0.39 -0.3 -0.5 rpy=0 0 3.14, axis -1 0 0, limit lower=0.0 upper=0.02 effort=1.0 velocity=1.5708, mimic joint=fridge_area_door_bottom_left_joint multiplier=0.01
- added joint fridge_area_door_top_left_handle_joint: type fixed, parent fridge_area_top_door, child fridge_area_top_door_handle, origin xyz=-0.036 -0.45 -0.65 rpy=1.57 0 0
- added joint fridge_area_door_top_left_joint: type revolute, parent fridge_area_door_top_out_fancy, child fridge_area_top_door, axis 0 0 -1, limit lower=0.0 upper=1.5708 effort=1000.0 velocity=1.5708
- added joint fridge_area_door_top_out_joint: type revolute, parent fridge_main, child fridge_area_door_top_out_fancy, origin xyz=0.39 -0.3 0.5 rpy=0 0 3.14, axis -1 0 0, limit lower=0.0 upper=1.5708 effort=1.0 velocity=1.5708, mimic joint=fridge_area_door_top_left_joint multiplier=0.01
- added joint fridge_area_joint: type fixed, parent side_A, child fridge_area, origin xyz=-0.273 1.022 1.07
- added joint fridge_back_joint: type fixed, parent fridge_main, child fridge_back, origin xyz=-0.1 0 0.4 rpy=0 0 0
- added joint fridge_bottom_side_joint: type fixed, parent fridge_main, child fridge_bottom_side, origin xyz=0.1 0. -0.2 rpy=0 0 0
- added joint fridge_left_side_joint: type fixed, parent fridge_main, child fridge_left_side, origin xyz=0.1 -0.25 0.4 rpy=0 0 -1.57
- added joint fridge_level1_joint: type fixed, parent fridge_main, child fridge_level1, origin xyz=0.1 0. 0.1 rpy=0 0 0
- added joint fridge_main_joint: type fixed, parent fridge_area, child fridge_main, origin xyz=0 0 0 rpy=0 0 0
- added joint fridge_right_side_joint: type fixed, parent fridge_main, child fridge_right_side, origin xyz=0.1 0.25 0.4 rpy=0 0 -1.57
- added joint fridge_top_side_joint: type fixed, parent fridge_main, child fridge_top_side, origin xyz=0.1 0. 1. rpy=0 0 0
- added joint island_left_bottom_handle_joint: type fixed, parent island_left_drawer_bottom, child island_left_bottom_handle, origin xyz=-0.24 0 0.245 rpy=1.57 0 0
- added joint island_left_drawer_bottom_joint: type prismatic, parent island_left, child island_left_drawer_bottom, origin xyz=0.036 0.0 -0.281 rpy=0 0 3.14, axis -1 0 0, limit lower=0.0 upper=0.45 effort=1000.0 velocity=0.5
- added joint island_left_drawer_middle_joint: type prismatic, parent island_left, child island_left_drawer_middle, origin xyz=0.027 0.0 0.106 rpy=0 0 3.14, axis -1 0 0, limit lower=0.0 upper=0.45 effort=1000.0 velocity=0.5
- added joint island_left_drawer_top_joint: type prismatic, parent island_left, child island_left_drawer_top, origin xyz=0.03 0.0 0.327 rpy=0 0 3.14, axis -1 0 0, limit lower=0.0 upper=0.45 effort=1000.0 velocity=0.5
- added joint island_left_joint: type fixed, parent side_B, child island_left, origin xyz=0.333 1.703 0.394
- added joint island_left_middle_handle_joint: type fixed, parent island_left_drawer_middle, child island_left_middle_handle, origin xyz=-0.245 0 0.13 rpy=1.57 0 0
- added joint island_left_top_handle_joint: type fixed, parent island_left_drawer_top, child island_left_top_handle, origin xyz=-0.245 0 0.05 rpy=1.57 0 0
- added joint island_middle_bottom_handle_joint: type fixed, parent island_middle_drawer_bottom, child island_middle_bottom_handle, origin xyz=-0.245 0 0.245 rpy=1.57 0 0
- added joint island_middle_drawer_bottom_joint: type prismatic, parent island_middle, child island_middle_drawer_bottom, origin xyz=0.03 0.0 -0.279 rpy=0 0 3.14, axis -1 0 0, limit lower=0.0 upper=0.45 effort=1000.0 velocity=0.5
- added joint island_middle_drawer_middle_joint: type prismatic, parent island_middle, child island_middle_drawer_middle, origin xyz=0.031 0.0 0.104 rpy=0 0 3.14, axis -1 0 0, limit lower=0.0 upper=0.45 effort=1000.0 velocity=0.5
- added joint island_middle_drawer_top_joint: type prismatic, parent island_middle, child island_middle_drawer_top, origin xyz=0.033 0.0 0.326 rpy=0 0 3.14, axis -1 0 0, limit lower=0.0 upper=0.45 effort=1000.0 velocity=0.5
- added joint island_middle_joint: type fixed, parent side_B, child island_middle, origin xyz=0.333 2.204 0.394
- added joint island_middle_middle_handle_joint: type fixed, parent island_middle_drawer_middle, child island_middle_middle_handle, origin xyz=-0.245 0 0.13 rpy=1.57 0 0
- added joint island_middle_top_handle_joint: type fixed, parent island_middle_drawer_top, child island_middle_top_handle, origin xyz=-0.243 0 0.05 rpy=1.57 0 0
- added joint island_right_bottom_handleott_joint: type fixed, parent island_right_drawer_bottom, child island_right_bottom_handle, origin xyz=-0.228 0 0.245 rpy=1.57 0 0
- added joint island_right_drawer_bottom_joint: type prismatic, parent island_right, child island_right_drawer_bottom, origin xyz=0.045 0.0 -0.286 rpy=0 0 3.14, axis -1 0 0, limit lower=0.0 upper=0.45 effort=1000.0 velocity=0.5
- added joint island_right_drawer_middle_joint: type prismatic, parent island_right, child island_right_drawer_middle, origin xyz=0.027 0.0 0.106 rpy=0 0 3.14, axis -1 0 0, limit lower=0.0 upper=0.45 effort=1000.0 velocity=0.5
- added joint island_right_drawer_top_joint: type prismatic, parent island_right, child island_right_drawer_top, origin xyz=0.03 0.0 0.326 rpy=0 0 3.14, axis -1 0 0, limit lower=0.0 upper=0.45 effort=1000.0 velocity=0.5
- added joint island_right_joint: type fixed, parent side_B, child island_right, origin xyz=0.333 2.855 0.394
- added joint island_right_middle_handle_joint: type fixed, parent island_right_drawer_middle, child island_right_middle_handle, origin xyz=-0.245 0 0.13 rpy=1.57 0 0
- added joint island_right_top_handle_joint: type fixed, parent island_right_drawer_top, child island_right_top_handle, origin xyz=-0.243 0 0.05 rpy=1.57 0 0
- added joint oven_area_coloksu_level4_joint: type fixed, parent oven_area, child oven_area_coloksu_level4, origin xyz=-0.172 0.005 0.281
- added joint oven_area_coloksu_level5_joint: type fixed, parent oven_area, child oven_area_coloksu_level5, origin xyz=-0.172 0.005 0.56
- added joint oven_area_door_top_left_handle_joint: type fixed, parent oven_area_door_top_left, child oven_area_door_top_left_handle, origin xyz=-0.055 -0.5 0.0 rpy=1.57 0 0
- added joint oven_area_door_top_left_joint: type revolute, parent oven_area, child oven_area_door_top_left, origin xyz=0.103 -0.3 0.32 rpy=0 0 3.14, axis 0 0 -1, limit lower=0.0 upper=1.5708 effort=1000.0 velocity=1.5708
- added joint oven_area_drawer_bottom_handle_joint: type fixed, parent oven_area_drawer_bottom, child oven_area_drawer_bottom_handle, origin xyz=-0.237 0.0 0.35 rpy=1.57 0 0
- added joint oven_area_drawer_bottom_joint: type prismatic, parent oven_area, child oven_area_drawer_bottom, origin xyz=-0.094 0.0 -0.95 rpy=0 0 3.14, axis -1 0 0, limit lower=0.0 upper=0.45 effort=1000.0 velocity=0.5
- added joint oven_area_drawer_middle_handle_joint: type fixed, parent oven_area_drawer_middle, child oven_area_drawer_middle_handle, origin xyz=-0.26 0.0 0.11 rpy=1.57 0 0
- added joint oven_area_drawer_middle_joint: type prismatic, parent oven_area, child oven_area_drawer_middle, origin xyz=-0.117 0.0 -0.43 rpy=0 0 3.14, axis -1 0 0, limit lower=0.0 upper=0.45 effort=1000.0 velocity=0.5
- added joint oven_area_joint: type fixed, parent side_A, child oven_area, origin xyz=0.01 0.01 1.02
- added joint oven_area_left_door_bottom_left_joint: type revolute, parent oven_area_left_door_bottom_out_fancy, child oven_area_left_door_bottom_left, axis 0 0 -1, limit lower=0.0 upper=1.5708 effort=1000.0 velocity=1.5708
- added joint oven_area_left_door_bottom_out_joint: type prismatic, parent oven_area_left, child oven_area_left_door_bottom_out_fancy, origin xyz=0.39 -0.3 -0.5 rpy=0 0 3.14, axis -1 0 0, limit lower=0.0 upper=0.02 effort=1.0 velocity=1.5708, mimic joint=oven_area_left_door_bottom_left_joint multiplier=0.01
- added joint oven_area_left_door_top_joint: type revolute, parent oven_area_left_door_top_out_fancy, child oven_area_left_door_top, axis 0 0 -1, limit lower=0.0 upper=1.5708 effort=1000.0 velocity=1.5708
- added joint oven_area_left_door_top_out_joint: type prismatic, parent oven_area_left, child oven_area_left_door_top_out_fancy, origin xyz=0.39 -0.3 0.5 rpy=0 0 3.14, axis -1 0 0, limit lower=0.0 upper=0.02 effort=1.0 velocity=1.5708, mimic joint=oven_area_left_door_top_joint multiplier=0.01
- added joint oven_area_left_joint: type fixed, parent side_A, child oven_area_left, origin xyz=-0.273 -0.5855 1.07
- added joint oven_area_right_door_left_joint: type revolute, parent oven_area_right_door_out_fancy, child oven_area_right_door, axis 0 0 -1, limit lower=0.0 upper=1.5708 effort=1000.0 velocity=1.5708
- added joint oven_area_right_door_out_joint: type prismatic, parent oven_area_right, child oven_area_right_door_out_fancy, origin xyz=0.277 -0.19 0.0 rpy=0 0 3.14, axis -1 0 0, limit lower=0.0 upper=0.02 effort=1.0 velocity=1.5708, mimic joint=oven_area_right_door_left_joint multiplier=0.01
- added joint oven_area_right_drawer_big_joint: type prismatic, parent oven_area_right, child oven_area_right_drawer_big, origin xyz=0.04 0.0 -0.12 rpy=0 0 3.14, axis -1 0 0, limit lower=0.0 upper=0.45 effort=500.0 velocity=0.5
- added joint oven_area_right_drawer_small_joint: type prismatic, parent oven_area_right, child oven_area_right_drawer_small, origin xyz=-0.01 0.0 0.17 rpy=0 0 3.14, axis -1 0 0, limit lower=0.0 upper=0.45 effort=500.0 velocity=0.5
- added joint oven_area_right_joint: type fixed, parent side_A, child oven_area_right, origin xyz=-0.163 0.51 0.975
- added joint sink_area_drawer_bottom_joint: type prismatic, parent sink_area, child sink_area_drawer_bottom, origin xyz=0.114 0.0 0.105 rpy=0 0 3.14, axis -1 0 0, limit lower=0.0 upper=0.45 effort=1000.0 velocity=0.5
- added joint sink_area_drawer_middle_joint: type prismatic, parent sink_area, child sink_area_drawer_middle, origin xyz=0.05 0.0 0.48 rpy=0 0 3.14, axis -1 0 0, limit lower=0.0 upper=0.40 effort=1000.0 velocity=0.5
- added joint sink_area_handle_top_joint: type fixed, parent sink_area_drawer_bottom, child sink_area_handle, origin xyz=-0.238 0 0.65 rpy=1.57 0 0
- added joint sink_area_joint: type fixed, parent side_B, child sink_area, origin xyz=0.256 1.102 0.006
- joint countertop_joint: parent cabinet5 -> coffee_area_bottom_left
- joint dishwasher_drawer_middle_joint: child dishwasher_drawer_middle -> dishwasher_drawer; parent cabinet7 -> dishwasher
- joint handle_cab2_drawer_bottom_joint: child handle_cab2_door -> oven_area_right_handle; parent cabinet2_door_left -> oven_area_right_door
- joint oven_joint: parent cabinet1 -> oven_area
- joint side_A_left_joint: origin xyz=-0.16 -0.296 1.030 rpy=0 0 1.57 -> xyz=-0.16 -0.896 1.030 rpy=0 0 1.57
